File: clock_2.kicad_pcb (KiCad board)
At the start: 2 copper layers, 82.8 x 84 mm, 68 parts, among them J1 VCC_DATA_GND, J2 VCC_DATA_GND

Commit message: aa
Parts:
- removed C1 (x4): 1000mF, Capacitors_THT:CP_Radial_D8.0mm_P3.80mm
- removed the J1 at (141.3, 107.1)
- removed the J1 at (98.3, 107.1)
- removed the J1 at (141.3, 64.1)
- removed the J2 at (108.4, 107.1)
- removed the J2 at (65.4, 107.1)
- removed the J2 at (108.4, 64.1)
- removed the LED1 at (132.8, 121.8)
- removed the LED1 at (89.8, 121.8)
- removed the LED1 at (132.8, 78.8)
- removed LED10 (x4), LED2 (x4), LED3 (x4), LED4 (x4), LED5 (x4), LED6 (x4), LED7 (x4), LED8 (x4), LED9 (x4): WS2812B, WS2812B:WS2812B
- removed the REF** at (107.7, 90.6)
- removed the REF** at (141.5, 125.6)
- removed the REF** at (98.5, 125.6)
- removed the REF** at (141.5, 82.6)
- removed the REF** at (64.7, 90.6)
- removed the REF** at (107.7, 47.6)
- removed the REF** at (141.5, 90.6)
- removed the REF** at (98.5, 90.6)
- removed the REF** at (141.5, 47.6)
- removed the REF** at (107.7, 125.6)
- removed the REF** at (64.7, 125.6)
- removed the REF** at (107.7, 82.6)
- moved LED1 12.2 mm to (89.8, 66.6), turned to 90 degrees
Connections:
- LED1 pad 2: Net-(LED1-Pad2) -> Net-(J2-Pad2)
Routing:
- net Net-(J1-Pad3): track 503.6 -> 43.2 mm
- net Net-(J1-Pad1): track 412.6 -> 38.1 mm
- net Net-(J1-Pad2): track 102.6 -> 6.80 mm
- net Net-(LED5-Pad2): track 73.7 -> 0.00 mm
- net Net-(LED2-Pad2): track 28.6 -> 0.00 mm
- net Net-(LED4-Pad2): track 27.6 -> 0.00 mm
- net Net-(LED1-Pad2): track 27.5 -> 0.00 mm
- net Net-(LED3-Pad2): track 27.4 -> 0.00 mm
- net Net-(LED8-Pad2): track 26.8 -> 0.00 mm
- net Net-(LED6-Pad2): track 26.5 -> 0.00 mm
- net Net-(LED7-Pad2): track 26.4 -> 0.00 mm
- net Net-(LED10-Pad4): track 26.3 -> 0.00 mm
- net Net-(J2-Pad2): track 52.9 -> 29.6 mm
Other:
- board size 82.8 x 84 mm -> 39.8 x 41 mm
- net class Default: trace_width 0.618 -> 0.9
